Commit message: add 2D Lidar sensor and scan visualization

File: src/roambot_description/urdf/roambot.urdf.xacro (robot description, xacro)
@@ -446,4 +446,47 @@
   </joint>
   <!-- ========================================================= -->
+  <!-- 2D LiDAR: distance sensor mounted above the front deck   -->
+  <!-- ========================================================= -->
+  <!-- Small circular mounting base resting on the upper deck -->
+  <link name="lidar_mount_link">
+    <visual>
+      <geometry>
+        <cylinder radius="0.033" length="0.006"/>
+      </geometry>
+      <material name="hub_dark_grey"/>
+    </visual>
+    <collision>
+      <geometry>
+        <cylinder radius="0.033" length="0.006"/>
+      </geometry>
+    </collision>
+    <xacro:cylinder_inertial mass="0.03" radius="0.033" length="0.006"/>
+  </link>
+  <joint name="lidar_mount_joint" type="fixed">
+    <parent link="base_link"/>
+    <child link="lidar_mount_link"/>
+    <origin xyz="0.075 0 0.0855" rpy="0 0 0"/>
+  </joint>
+  <!-- LiDAR housing raised above its mounting base -->
+  <link name="lidar_link">
+    <visual>
+      <geometry>
+        <cylinder radius="0.025" length="0.025"/>
+      </geometry>
+      <material name="hub_dark_grey"/>
+    </visual>
+    <collision>
+      <geometry>
+        <cylinder radius="0.025" length="0.025"/>
+      </geometry>
+    </collision>
+    <xacro:cylinder_inertial mass="0.06" radius="0.025" length="0.025"/>
+  </link>
+  <joint name="lidar_joint" type="fixed">
+    <parent link="lidar_mount_link"/>
+    <child link="lidar_link"/>
+    <origin xyz="0 0 0.0155" rpy="0 0 0"/>
+  </joint>
+  <!-- ========================================================= -->
   <!-- Gazebo physical properties                                -->
   <!-- ========================================================= -->
@@ -461,4 +504,28 @@
     <mu1>0.15</mu1>
     <mu2>0.15</mu2>
+  </gazebo>
+  <gazebo reference="lidar_link">
+    <sensor name="lidar_sensor" type="gpu_lidar">
+      <pose>0 0 0 0 0 0</pose>
+      <topic>/model/roambot/scan</topic>
+      <update_rate>10</update_rate>
+      <always_on>true</always_on>
+      <visualize>false</visualize>
+      <lidar>
+        <scan>
+          <horizontal>
+            <samples>360</samples>
+            <resolution>1</resolution>
+            <min_angle>-3.14159</min_angle>
+            <max_angle>3.14159</max_angle>
+          </horizontal>
+        </scan>
+        <range>
+          <min>0.12</min>
+          <max>6.0</max>
+          <resolution>0.01</resolution>
+        </range>
+      </lidar>
+    </sensor>
   </gazebo>
     <!-- Gazebo's built-in differential-drive controller -->

Commit message: parameterize roambot model for multi-robot simulation

File: src/roambot_description/urdf/roambot.urdf.xacro (robot description, xacro)
@@ -1,4 +1,9 @@
 <?xml version="1.0"?>
 <robot xmlns:xacro="http://www.ros.org/wiki/xacro" name="roambot">
+  <!-- Values used when multiple RoamBots are spawned in one world. -->
+  <xacro:arg name="model_name" default="roambot"/>
+  <xacro:arg name="frame_prefix" default=""/>
+  <xacro:property name="model_name" value="$(arg model_name)"/>
+  <xacro:property name="frame_prefix" value="$(arg frame_prefix)"/>
   <!-- ========================================================= -->
   <!-- TRI-ROVER: Concept 2WD differential-drive mobile robot    -->
@@ -508,5 +513,5 @@
     <sensor name="lidar_sensor" type="gpu_lidar">
       <pose>0 0 0 0 0 0</pose>
-      <topic>/model/roambot/scan</topic>
+      <topic>/model/${model_name}/scan</topic>
       <update_rate>10</update_rate>
       <always_on>true</always_on>
@@ -540,10 +545,10 @@
       <wheel_radius>0.065</wheel_radius>
       <!-- Gazebo topic names -->
-      <topic>/model/roambot/cmd_vel</topic>
-      <odom_topic>/model/roambot/odometry</odom_topic>
-      <tf_topic>/model/roambot/tf</tf_topic>
+      <topic>/model/${model_name}/cmd_vel</topic>
+      <odom_topic>/model/${model_name}/odometry</odom_topic>
+      <tf_topic>/model/${model_name}/tf</tf_topic>
       <!-- Names used inside odometry messages -->
-      <frame_id>odom</frame_id>
-      <child_frame_id>base_footprint</child_frame_id>
+      <frame_id>${frame_prefix}odom</frame_id>
+      <child_frame_id>${frame_prefix}base_footprint</child_frame_id>
       <!-- Publish 30 position updates per second -->
       <odom_publish_frequency>30</odom_publish_frequency>
@@ -557,5 +562,5 @@
     <plugin filename="gz-sim-joint-state-publisher-system"
             name="gz::sim::systems::JointStatePublisher">
-      <topic>/model/roambot/joint_states</topic>
+      <topic>/model/${model_name}/joint_states</topic>
       <joint_name>left_wheel_joint</joint_name>
       <joint_name>right_wheel_joint</joint_name>

Commit message: add scout camera inventory tag detection

File: src/roambot_description/urdf/roambot.urdf.xacro (robot description, xacro)
@@ -4,11 +4,11 @@
   <xacro:arg name="model_name" default="roambot"/>
   <xacro:arg name="frame_prefix" default=""/>
+  <xacro:property name="enable_camera" value="$(arg enable_camera)"/>
   <xacro:property name="model_name" value="$(arg model_name)"/>
   <xacro:property name="frame_prefix" value="$(arg frame_prefix)"/>
-  <!-- ========================================================= -->
+  <xacro:property name="enable_camera" value="$(arg enable_camera)"/>
   <!-- TRI-ROVER: Concept 2WD differential-drive mobile robot    -->
   <!-- Simplified physical model designed for ROS 2 / Gazebo     -->
   <!-- Units: SI (meters, kilograms, radians)                     -->
-  <!-- ========================================================= -->
   <!-- - Parameters - -->
   <xacro:property name="body_length" value="0.30"/>
@@ -92,7 +92,8 @@
     <color rgba="0.26 0.28 0.30 1.0"/>
   </material>
-  <!-- ========================================================= -->
-  <!-- Helper macros                                              -->
-  <!-- ========================================================= -->
+  <material name="camera_lens_silver">
+    <color rgba="0.78 0.80 0.82 1.0"/>
+  </material>
+  <!-- Helper macros-->
   <xacro:macro name="box_inertial" params="mass x y z">
     <inertial>
@@ -148,7 +149,5 @@
     </joint>
   </xacro:macro>
-  <!-- ========================================================= -->
-  <!-- Base frame                                                 -->
-  <!-- ========================================================= -->
+  <!-- Base frame-->
   <link name="base_footprint"/>
   <joint name="base_footprint_joint" type="fixed">
@@ -157,7 +156,5 @@
     <origin xyz="0 0 ${body_z}" rpy="0 0 0"/>
   </joint>
-  <!-- ========================================================= -->
-  <!-- Main chassis                                               -->
-  <!-- ========================================================= -->
+  <!-- Main chassis-->
   <link name="base_link">
     <!--
@@ -221,7 +218,5 @@
   <xacro:standoff_pillar name="rear_pillar"
                          x="${pillar_rear_x}" y="${pillar_rear_y}"/>
-  <!-- ========================================================= -->
   <!-- Upper wedge deck                                           -->
-  <!-- ========================================================= -->
   <link name="upper_deck">
     <!--
@@ -313,8 +308,6 @@
             rpy="0 0 0"/>
   </joint>
-  <!-- ========================================================= -->
-  <!-- Drive wheels                                               -->
+  <!-- Drive wheels-->
   <!-- Cylinder axis is rotated to align with robot Y-axis       -->
-  <!-- ========================================================= -->
   <link name="left_wheel_link">
     <visual>
@@ -361,9 +354,7 @@
     <axis xyz="0 1 0"/>
   </joint>
-  <!-- ========================================================= -->
   <!-- Rear caster assembly                                      -->
   <!-- Fork is fixed to chassis; caster wheel rotates freely     -->
   <!-- Wheel bottom is aligned to z = 0 ground plane             -->
-  <!-- ========================================================= -->
   <link name="caster_mount_link">
     <visual>
@@ -450,7 +441,5 @@
     <dynamics damping="0.02" friction="0.01"/>
   </joint>
-  <!-- ========================================================= -->
   <!-- 2D LiDAR: distance sensor mounted above the front deck   -->
-  <!-- ========================================================= -->
   <!-- Small circular mounting base resting on the upper deck -->
   <link name="lidar_mount_link">
@@ -493,7 +482,31 @@
     <origin xyz="0 0 0.0155" rpy="0 0 0"/>
   </joint>
-  <!-- ========================================================= -->
+  <!-- Optional front camera for visual inventory inspection      -->
+  <xacro:if value="${enable_camera}">
+    <link name="camera_link">
+      <visual>
+        <geometry>
+          <box size="0.040 0.050 0.030"/>
+        </geometry>
+        <material name="hub_dark_grey"/>
+      </visual>
+      <!-- Lens faces RoamBot's forward (+X) direction -->
+      <visual>
+        <origin xyz="0.021 0 0" rpy="0 ${pi/2} 0"/>
+        <geometry>
+          <cylinder radius="0.011" length="0.010"/>
+        </geometry>
+        <material name="camera_lens_silver"/>
+      </visual>
+      <xacro:box_inertial mass="0.04" x="0.040" y="0.050" z="0.030"/>
+    </link>
+    <joint name="camera_joint" type="fixed">
+      <parent link="base_link"/>
+      <child link="camera_link"/>
+      <!-- +X is RoamBot's forward direction -->
+      <origin xyz="0.130 0 0.0375" rpy="0 0 0"/>
+    </joint>
+  </xacro:if>
   <!-- Gazebo physical properties                                -->
-  <!-- ========================================================= -->
   <gazebo reference="base_link">
   </gazebo>
@@ -534,4 +547,28 @@
     </sensor>
   </gazebo>
+  <xacro:if value="${enable_camera}">
+    <gazebo reference="camera_link">
+      <sensor name="inventory_camera" type="camera">
+        <pose>0 0 0 0 0 0</pose>
+        <topic>/model/${model_name}/camera/image</topic>
+        <update_rate>10</update_rate>
+        <always_on>true</always_on>
+        <visualize>false</visualize>
+        <camera>
+          <horizontal_fov>1.047</horizontal_fov>
+          <image>
+            <width>640</width>
+            <height>480</height>
+            <format>R8G8B8</format>
+          </image>
+          <clip>
+            <near>0.05</near>
+            <far>5.0</far>
+          </clip>
+          <camera_info_topic>/model/${model_name}/camera/camera_info</camera_info_topic>
+        </camera>
+      </sensor>
+    </gazebo>
+  </xacro:if>
     <!-- Gazebo's built-in differential-drive controller -->
   <gazebo>
