Commit message: rebuild warehouse navigation and add visual tag alignment

File: src/roambot_description/urdf/roambot.urdf.xacro (robot description, xacro)
@@ -1,99 +1,36 @@
 <?xml version="1.0"?>
 <robot xmlns:xacro="http://www.ros.org/wiki/xacro" name="roambot">
-  <!-- Values used when multiple RoamBots are spawned in one world. -->
   <xacro:arg name="model_name" default="roambot"/>
   <xacro:arg name="frame_prefix" default=""/>
-  <xacro:property name="enable_camera" value="$(arg enable_camera)"/>
+  <xacro:arg name="enable_camera" default="false"/>
   <xacro:property name="model_name" value="$(arg model_name)"/>
   <xacro:property name="frame_prefix" value="$(arg frame_prefix)"/>
   <xacro:property name="enable_camera" value="$(arg enable_camera)"/>
-  <!-- TRI-ROVER: Concept 2WD differential-drive mobile robot    -->
-  <!-- Simplified physical model designed for ROS 2 / Gazebo     -->
-  <!-- Units: SI (meters, kilograms, radians)                     -->
-  <!-- - Parameters - -->
-  <xacro:property name="body_length" value="0.30"/>
-  <xacro:property name="body_width"  value="0.22"/>
-  <xacro:property name="body_height" value="0.045"/>
-  <xacro:property name="upper_length" value="0.255"/>
-  <xacro:property name="upper_width"  value="0.175"/>
-  <xacro:property name="upper_height" value="0.020"/>
-  <!-- Three standoff pillars matching the reversed triangular upper deck -->
-  <xacro:property name="pillar_radius" value="0.008"/>
-  <xacro:property name="pillar_height" value="0.040"/>
-  <!-- Two front corner pillars -->
-  <xacro:property name="pillar_front_x" value="0.070"/>
-  <xacro:property name="pillar_front_y" value="0.060"/>
-  <!-- One rear pillar centred below the short rear edge -->
-  <xacro:property name="pillar_rear_x" value="-0.090"/>
-  <xacro:property name="pillar_rear_y" value="0.000"/>
-  <!-- Capsule-shaped chassis: straight sides + rounded front + rounded rear -->
-  <xacro:property name="chassis_width" value="0.205"/>
-  <xacro:property name="chassis_total_length" value="0.300"/>
-  <xacro:property name="chassis_round_radius" value="${chassis_width / 2.0}"/>
-  <!-- Distance between the two rounded-end centres -->
-  <xacro:property name="chassis_straight_length"
-                  value="${chassis_total_length - 2.0 * chassis_round_radius}"/>
-  <!-- Front and rear circle centres -->
-  <xacro:property name="chassis_front_x"
-                  value="${chassis_straight_length / 2.0}"/>
-  <xacro:property name="chassis_rear_x"
-                  value="${-chassis_straight_length / 2.0}"/>
-  <!-- Primitive-only clipped triangular upper deck -->
-  <xacro:property name="deck_rail_width" value="0.030"/>
-  <!-- Outer corner centres -->
-  <xacro:property name="deck_front_x" value="0.075"/>
-  <xacro:property name="deck_front_y" value="0.065"/>
-  <xacro:property name="deck_rear_x" value="-0.095"/>
-  <xacro:property name="deck_rear_y" value="0.025"/>
-  <!-- Rail geometry -->
-  <xacro:property name="deck_front_rail_length" value="0.130000"/>
-  <xacro:property name="deck_rear_rail_length" value="0.050000"/>
-  <xacro:property name="deck_side_rail_length" value="0.174642"/>
-  <xacro:property name="deck_left_mid_x" value="-0.010000"/>
-  <xacro:property name="deck_left_mid_y" value="0.045000"/>
-  <xacro:property name="deck_right_mid_x" value="-0.010000"/>
-  <xacro:property name="deck_right_mid_y" value="-0.045000"/>
-  <xacro:property name="deck_left_rail_yaw" value="-2.91050199"/>
-  <xacro:property name="deck_right_rail_yaw" value="2.91050199"/>
-  <!-- Corner cap radius hides square-ended rail intersections -->
-  <xacro:property name="deck_corner_radius" value="${deck_rail_width / 2.0}"/>
-  <xacro:property name="wheel_radius" value="0.065"/>
-  <xacro:property name="wheel_width"  value="0.030"/>
-  <!-- Drive wheel centreline: inner tire face touches chassis outer face -->
-  <xacro:property name="wheel_y"
-                  value="${chassis_width / 2.0 + wheel_width / 2.0}"/>
-  <xacro:property name="wheel_x"      value="0.030"/>
-  <xacro:property name="caster_radius" value="0.022"/>
-  <xacro:property name="caster_width"  value="0.016"/>
-  <xacro:property name="caster_x"      value="-0.115"/>
-  <!-- Main chassis bottom is intentionally above wheel contact plane -->
-  <xacro:property name="body_z" value="0.070"/>
-  <!-- - Materials - -->
-  <!-- Main color palette -->
-  <material name="chassis_metallic_green">
-    <color rgba="0.12 0.34 0.20 1.0"/>
-  </material>
-  <material name="deck_olive">
-    <color rgba="0.28 0.34 0.23 1.0"/>
-  </material>
-  <material name="panel_light_grey">
-    <color rgba="0.72 0.74 0.76 1.0"/>
-  </material>
-  <material name="wheel_light_brown">
-    <color rgba="0.58 0.36 0.20 1.0"/>
-  </material>
-  <material name="caster_silver">
-    <color rgba="0.78 0.80 0.82 1.0"/>
-  </material>
-  <material name="pillar_gold">
-    <color rgba="0.83 0.62 0.12 1.0"/>
-  </material>
-  <material name="hub_dark_grey">
-    <color rgba="0.26 0.28 0.30 1.0"/>
-  </material>
-  <material name="camera_lens_silver">
-    <color rgba="0.78 0.80 0.82 1.0"/>
-  </material>
-  <!-- Helper macros-->
+  <!-- Four-wheel chassis: 0.66 m long, 0.51 m wide including the wheels. -->
+  <xacro:property name="body_length" value="0.70"/>
+  <xacro:property name="body_width" value="0.42"/>
+  <xacro:property name="body_height" value="0.08"/>
+  <xacro:property name="body_z" value="0.12"/>
+  <xacro:property name="body_round_radius" value="${body_width / 2.0}"/>
+  <xacro:property name="body_straight_length" value="${body_length - 2.0 * body_round_radius}"/>
+  <xacro:property name="body_end_x" value="${body_straight_length / 2.0}"/>
+  <xacro:property name="wheel_radius" value="0.075"/>
+  <xacro:property name="wheel_width" value="0.045"/>
+  <xacro:property name="wheel_y" value="${body_width / 2.0 + wheel_width / 2.0}"/>
+  <xacro:property name="front_wheel_x" value="0.20"/>
+  <xacro:property name="rear_wheel_x" value="-0.20"/>
+  <xacro:property name="wheel_z" value="${-body_z + wheel_radius}"/>
+  <xacro:property name="deck_height" value="0.03"/>
+  <xacro:property name="pillar_height" value="0.07"/>
+  <xacro:property name="pillar_radius" value="0.014"/>
+  <!-- Original RoamBot colour palette. -->
+  <material name="body_color"><color rgba="0.12 0.34 0.20 1"/></material>
+  <material name="deck_color"><color rgba="0.28 0.34 0.23 1"/></material>
+  <material name="metal"><color rgba="0.72 0.74 0.76 1"/></material>
+  <material name="dark_metal"><color rgba="0.26 0.28 0.30 1"/></material>
+  <material name="wheel_color"><color rgba="0.58 0.36 0.20 1"/></material>
+  <material name="pillar_gold"><color rgba="0.83 0.62 0.12 1"/></material>
+  <material name="camera_lens_silver"><color rgba="0.78 0.80 0.82 1"/></material>
+  <material name="tote_color"><color rgba="0.30 0.34 0.38 1"/></material>
   <xacro:macro name="box_inertial" params="mass x y z">
     <inertial>
@@ -101,9 +38,6 @@
       <origin xyz="0 0 0"/>
       <inertia
-        ixx="${mass * (y*y + z*z) / 12.0}"
-        ixy="0.0"
-        ixz="0.0"
-        iyy="${mass * (x*x + z*z) / 12.0}"
-        iyz="0.0"
+        ixx="${mass * (y*y + z*z) / 12.0}" ixy="0" ixz="0"
+        iyy="${mass * (x*x + z*z) / 12.0}" iyz="0"
         izz="${mass * (x*x + y*y) / 12.0}"/>
     </inertial>
@@ -114,416 +48,349 @@
       <origin xyz="0 0 0"/>
       <inertia
-        ixx="${mass * (3*radius*radius + length*length) / 12.0}"
-        ixy="0.0"
-        ixz="0.0"
-        iyy="${mass * (3*radius*radius + length*length) / 12.0}"
-        iyz="0.0"
+        ixx="${mass * (3*radius*radius + length*length) / 12.0}" ixy="0" ixz="0"
+        iyy="${mass * (3*radius*radius + length*length) / 12.0}" iyz="0"
         izz="${mass * radius*radius / 2.0}"/>
     </inertial>
   </xacro:macro>
-  <!-- Reusable structural standoff pillar -->
-  <xacro:macro name="standoff_pillar" params="name x y">
+  <link name="base_footprint"/>
+  <joint name="base_footprint_joint" type="fixed">
+    <parent link="base_footprint"/>
+    <child link="base_link"/>
+    <origin xyz="0 0 ${body_z}"/>
+  </joint>
+  <!-- Rounded, longer mobile base. The box and end cylinders form a capsule. -->
+  <link name="base_link">
+    <visual>
+      <geometry><box size="${body_straight_length} ${body_width} ${body_height}"/></geometry>
+      <material name="body_color"/>
+    </visual>
+    <visual>
+      <origin xyz="${body_end_x} 0 0"/>
+      <geometry><cylinder radius="${body_round_radius}" length="${body_height}"/></geometry>
+      <material name="body_color"/>
+    </visual>
+    <visual>
+      <origin xyz="${-body_end_x} 0 0"/>
+      <geometry><cylinder radius="${body_round_radius}" length="${body_height}"/></geometry>
+      <material name="body_color"/>
+    </visual>
+    <collision>
+      <geometry><box size="${body_straight_length} ${body_width} ${body_height}"/></geometry>
+    </collision>
+    <collision>
+      <origin xyz="${body_end_x} 0 0"/>
+      <geometry><cylinder radius="${body_round_radius}" length="${body_height}"/></geometry>
+    </collision>
+    <collision>
+      <origin xyz="${-body_end_x} 0 0"/>
+      <geometry><cylinder radius="${body_round_radius}" length="${body_height}"/></geometry>
+    </collision>
+    <xacro:box_inertial mass="10.0" x="${body_length}" y="${body_width}" z="${body_height}"/>
+  </link>
+  <!-- Low triangular deck above the chassis. -->
+  <link name="upper_deck_link">
+    <visual>
+      <geometry><box size="0.38 0.30 ${deck_height}"/></geometry>
+      <material name="deck_color"/>
+    </visual>
+    <visual>
+      <origin xyz="0.17 0 0.025"/>
+      <geometry><box size="0.05 0.30 0.04"/></geometry>
+      <material name="metal"/>
+    </visual>
+    <xacro:box_inertial mass="1.1" x="0.38" y="0.30" z="${deck_height}"/>
+  </link>
+  <joint name="upper_deck_joint" type="fixed">
+    <parent link="base_link"/>
+    <child link="upper_deck_link"/>
+    <origin xyz="0 0 ${body_height / 2.0 + pillar_height + deck_height / 2.0}"/>
+  </joint>
+  <xacro:macro name="deck_pillar" params="name x y">
     <link name="${name}_link">
       <visual>
-        <origin xyz="0 0 0"/>
-        <geometry>
-          <cylinder radius="${pillar_radius}" length="${pillar_height}"/>
-        </geometry>
+        <geometry><cylinder radius="${pillar_radius}" length="${pillar_height}"/></geometry>
         <material name="pillar_gold"/>
       </visual>
-      <collision>
-        <origin xyz="0 0 0"/>
-        <geometry>
-          <cylinder radius="${pillar_radius}" length="${pillar_height}"/>
-        </geometry>
-      </collision>
-      <xacro:cylinder_inertial
-        mass="0.035"
-        radius="${pillar_radius}"
-        length="${pillar_height}"/>
+      <xacro:cylinder_inertial mass="0.06" radius="${pillar_radius}" length="${pillar_height}"/>
     </link>
     <joint name="${name}_joint" type="fixed">
       <parent link="base_link"/>
       <child link="${name}_link"/>
-      <origin xyz="${x} ${y} ${body_height/2 + pillar_height/2}" rpy="0 0 0"/>
+      <origin xyz="${x} ${y} ${body_height / 2.0 + pillar_height / 2.0}"/>
     </joint>
   </xacro:macro>
-  <!-- Base frame-->
-  <link name="base_footprint"/>
-  <joint name="base_footprint_joint" type="fixed">
-    <parent link="base_footprint"/>
-    <child link="base_link"/>
-    <origin xyz="0 0 ${body_z}" rpy="0 0 0"/>
-  </joint>
-  <!-- Main chassis-->
-  <link name="base_link">
-    <!--
-      Straight middle section.
-      Its side faces are parallel to the drive wheels.
-    -->
-    <visual>
-      <origin xyz="0 0 0"/>
-      <geometry>
-        <box size="${chassis_straight_length} ${chassis_width} ${body_height}"/>
-      </geometry>
-      <material name="chassis_metallic_green"/>
-    </visual>
-    <!-- Rounded front end -->
-    <visual>
-      <origin xyz="${chassis_front_x} 0 0"/>
-      <geometry>
-        <cylinder radius="${chassis_round_radius}" length="${body_height}"/>
-      </geometry>
-      <material name="chassis_metallic_green"/>
-    </visual>
-    <!-- Rounded rear end -->
-    <visual>
-      <origin xyz="${chassis_rear_x} 0 0"/>
-      <geometry>
-        <cylinder radius="${chassis_round_radius}" length="${body_height}"/>
-      </geometry>
-      <material name="chassis_metallic_green"/>
-    </visual>
-    <!-- Collision geometry mirrors the simple capsule construction -->
+  <xacro:deck_pillar name="front_left_pillar" x="0.14" y="0.11"/>
+  <xacro:deck_pillar name="front_right_pillar" x="0.14" y="-0.11"/>
+  <xacro:deck_pillar name="rear_pillar" x="-0.16" y="0"/>
+  <!--
+    Tote carrier chain
+    base_link -> lift_mast_link -> lift_carriage_link -> tote_slide_link -> carried_tote_link
+    The tray is supported by the carriage, not placed in mid-air.
+  -->
+  <link name="lift_mast_link">
+    <visual>
+      <origin xyz="0 0.07 0"/>
+      <geometry><box size="0.055 0.030 0.76"/></geometry>
+      <material name="metal"/>
+    </visual>
+    <visual>
+      <origin xyz="0 -0.07 0"/>
+      <geometry><box size="0.055 0.030 0.76"/></geometry>
+      <material name="metal"/>
+    </visual>
+    <visual>
+      <origin xyz="0 0 0.325"/>
+      <geometry><box size="0.060 0.17 0.05"/></geometry>
+      <material name="dark_metal"/>
+    </visual>
+    <visual>
+      <origin xyz="0 0 -0.325"/>
+      <geometry><box size="0.070 0.18 0.07"/></geometry>
+      <material name="dark_metal"/>
+    </visual>
+    <xacro:box_inertial mass="1.8" x="0.07" y="0.18" z="0.76"/>
+  </link>
+  <joint name="lift_mast_joint" type="fixed">
+    <parent link="base_link"/>
+    <child link="lift_mast_link"/>
+    <origin xyz="-0.16 0 0.52"/>
+  </joint>
+  <!--
+    The carrier starts on the upper-deck surface.  Every carriage and tray
+    visual begins at z=0 or above, so no part enters the deck at lift=0.
+  -->
+  <link name="lift_carriage_link">
+    <!-- Two guide shoes visibly lock the carriage to the mast rails. -->
+    <visual>
+      <origin xyz="0 0.070 0.055"/>
+      <geometry><box size="0.090 0.060 0.110"/></geometry>
+      <material name="metal"/>
+    </visual>
+    <visual>
+      <origin xyz="0 -0.070 0.055"/>
+      <geometry><box size="0.090 0.060 0.110"/></geometry>
+      <material name="metal"/>
+    </visual>
+    <!-- A cross-head joins the guide shoes; it remains part of the mast. -->
+    <visual>
+      <origin xyz="0 0 0.055"/>
+      <geometry><box size="0.090 0.180 0.060"/></geometry>
+      <material name="dark_metal"/>
+    </visual>
+    <!-- Narrow fixed rails support the sliding tray at the same deck level. -->
+    <visual>
+      <origin xyz="0.260 0.130 0.020"/>
+      <geometry><box size="0.440 0.030 0.040"/></geometry>
+      <material name="dark_metal"/>
+    </visual>
+    <visual>
+      <origin xyz="0.260 -0.130 0.020"/>
+      <geometry><box size="0.440 0.030 0.040"/></geometry>
+      <material name="dark_metal"/>
+    </visual>
+    <visual>
+      <origin xyz="0.070 0 0.020"/>
+      <geometry><box size="0.040 0.290 0.040"/></geometry>
+      <material name="dark_metal"/>
+    </visual>
+    <xacro:box_inertial mass="1.2" x="0.53" y="0.29" z="0.12"/>
+  </link>
+  <joint name="lift_joint" type="prismatic">
+    <parent link="lift_mast_link"/>
+    <child link="lift_carriage_link"/>
+    <origin xyz="0 0 -0.38"/>
+    <axis xyz="0 0 1"/>
+    <limit lower="0.0" upper="0.56" effort="350" velocity="0.18"/>
+    <dynamics damping="30" friction="3"/>
+  </joint>
+  <!-- The tray sits on the same plane as the fixed carriage rails. -->
+  <link name="tote_slide_link">
+    <visual>
+      <origin xyz="0.220 0 0.020"/>
+      <geometry><box size="0.400 0.240 0.040"/></geometry>
+      <material name="metal"/>
+    </visual>
+    <visual>
+      <origin xyz="0.220 0.1125 0.075"/>
+      <geometry><box size="0.400 0.015 0.110"/></geometry>
+      <material name="dark_metal"/>
+    </visual>
+    <visual>
+      <origin xyz="0.220 -0.1125 0.075"/>
+      <geometry><box size="0.400 0.015 0.110"/></geometry>
+      <material name="dark_metal"/>
+    </visual>
+    <visual>
+      <origin xyz="0.035 0 0.075"/>
+      <geometry><box size="0.015 0.240 0.110"/></geometry>
+      <material name="dark_metal"/>
+    </visual>
+    <xacro:box_inertial mass="0.8" x="0.400" y="0.240" z="0.13"/>
+  </link>
+  <joint name="tote_slide_joint" type="prismatic">
+    <parent link="lift_carriage_link"/>
+    <child link="tote_slide_link"/>
+    <origin xyz="0.080 0 0"/>
+    <axis xyz="1 0 0"/>
+    <limit lower="0.0" upper="0.20" effort="250" velocity="0.14"/>
+    <dynamics damping="25" friction="2"/>
+  </joint>
+  <!-- A neutral tote stays seated on the tray and demonstrates the full mechanism. -->
+  <link name="carried_tote_link">
+    <visual>
+      <origin xyz="0.220 0 0.055"/>
+      <geometry><box size="0.26 0.17 0.015"/></geometry>
+      <material name="tote_color"/>
+    </visual>
+    <visual>
+      <origin xyz="0.220 0.0775 0.1075"/>
+      <geometry><box size="0.26 0.015 0.100"/></geometry>
+      <material name="tote_color"/>
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